File: electrical/edge_io_rings/kicad/edge_io_rings.kicad_sch (KiCad schematic)
At the start: 12 parts, among them U1 nRF52840-QIAA-R, U10 TLV70033DSET, U2 BMI270, U3 IQS7222A, U4 DWM3001C, U5 BHI360, U6 BMM350, U7 SE050C1HQ1, U8 DRV2605LDGSR, U9 BQ25100YFPR

Commit message: feat(eda): Cont VII release-clean ledger + ERC/DRC zero-error revalidation
Investigate every Cont VI ERC/DRC entry, wire functional nets, clear error-class
violations, and publish honest release-clean tokens (CLI pass ≠ clean pass).

Co-authored-by: Cursor <cursoragent@cursor.com>
Parts:
- removed ANT1: 2450AT18A100, symbol Device:R
- removed BT1: LiPo_80to250mAh, symbol Device:R
- removed U1: nRF52840-QIAA-R, symbol Device:R
- removed U10: TLV70033DSET, symbol Device:R
- removed U2: BMI270, symbol Device:R
- removed U3: IQS7222A, symbol Device:R
- removed U4: DWM3001C, module, symbol Device:R
- removed U5: BHI360, symbol Device:R
- removed U6: BMM350, symbol Device:R
- removed U7: SE050C1HQ1, symbol Device:R
- removed U8: DRV2605LDGSR, symbol Device:R
- removed U9: BQ25100YFPR, symbol Device:R
- added ANT1: 2450AT18A100, gunnchos_structural:Block_SMD_10x10, symbol FuncBlock
- added BT1: LiPo_80to250mAh, gunnchos_structural:Block_SMD_10x10, symbol FuncBlock
- added U1: nRF52840-QIAA-R, gunnchos_structural:Block_SMD_10x10, symbol FuncBlock
- added U10: TLV75533PDBVR, gunnchos_structural:Block_SMD_10x10, symbol FuncBlock
- added U2: BMI270, gunnchos_structural:Block_SMD_10x10, symbol FuncBlock
- added U3: IQS7222A, gunnchos_structural:Block_SMD_10x10, symbol FuncBlock
- added U4: DWM3001C, gunnchos_structural:Block_SMD_10x10, symbol FuncBlock
- added U5: BHI360, gunnchos_structural:Block_SMD_10x10, symbol FuncBlock
- added U6: BMM350, gunnchos_structural:Block_SMD_10x10, symbol FuncBlock
- added U7: SE050C1HQ1, gunnchos_structural:Block_SMD_10x10, symbol FuncBlock
- added U8: DRV2605LDGSR, gunnchos_structural:Block_SMD_10x10, symbol FuncBlock
- added U9: npm1300-CAAA-R, gunnchos_structural:Block_SMD_10x10, symbol FuncBlock
Connections:
- net CAP_RDY: now also U10.2
- net I2C_SCL: now also U3.2
- net I2C_SDA: now also U2.2
- net IMU_INT: now also U5.2
- net SPI_UWB: now also U4.2
- net VDD_3V3: now also U1.2
- new net CHG_STATUS: U8.2
- new net HAPTIC_TRIG: U9.2
- new net SE_I2C_SCL: U7.2
- new net SE_I2C_SDA: U6.2
- no-connect marks 0 -> 14
Other:
- company: gunnchOS3k / HARDWARE FAMILY DEPTH -> gunnchOS3k / CONTINUATION VII
- title: Edge I/O Ring EVT1 — ADR-FP-008 fusion -> Edge I/O Ring EVT1 — Cont VII
