File: electrical/handheld_hybrid/kicad/handheld_hybrid.kicad_sch (KiCad schematic)
At the start: 11 parts

Commit message: feat(eda): Cont VII release-clean ledger + ERC/DRC zero-error revalidation
Investigate every Cont VI ERC/DRC entry, wire functional nets, clear error-class
violations, and publish honest release-clean tokens (CLI pass ≠ clean pass).

Co-authored-by: Cursor <cursoragent@cursor.com>
Parts:
- removed BT1: 6000mAh_pack, symbol Device:R
- removed J_DISP: 7in_1080p_120Hz, symbol Device:R
- removed J_USBC: USB_C_DP_Alt, symbol Device:R
- removed USOM1: RM121-D8E32, symbol Device:R
- removed U_CHG: BQ25895_or_BQ25792, symbol Device:R
- removed U_FG: BQ27Z273, symbol Device:R
- removed U_HID: STM32F103C8T6, symbol Device:R
- removed U_PD: TPS65987_or_IP2726, symbol Device:R
- removed U_SE: SE050C1HQ1, symbol Device:R
- removed U_WIFI: AP6275P_or_AIC8800D, symbol Device:R
- removed U_WWAN: RM520N-GL, symbol Device:R
- added BT1: 6000mAh_pack, gunnchos_structural:Block_SMD_10x10, symbol FuncBlock
- added JS1, JS2: RKJXV122400D, gunnchos_structural:Block_SMD_10x10, symbol FuncBlock
- added JSOM1: SODIMM-260, gunnchos_structural:Block_SMD_10x10, symbol FuncBlock
- added J_AUDIO: I2S_HP_codec, gunnchos_structural:Block_SMD_10x10, symbol FuncBlock
- added J_DBG: UART2_3pin, gunnchos_structural:Block_SMD_10x10, symbol FuncBlock
- added J_DISP: 7in_1080p_120Hz_IPS, gunnchos_structural:Block_SMD_10x10, symbol FuncBlock
- added J_USBC: USB_C_receptacle, gunnchos_structural:Block_SMD_10x10, symbol FuncBlock
- added J_USD: microSD_socket, gunnchos_structural:Block_SMD_10x10, symbol FuncBlock
- added SW_ABXY: tactile_ABXY_LR_DPAD, gunnchos_structural:Block_SMD_10x10, symbol FuncBlock
- added USOM1: RM121-D8E32, gunnchos_structural:Block_SMD_10x10, symbol FuncBlock
- added U_CHG: BQ25895RTWR, gunnchos_structural:Block_SMD_10x10, symbol FuncBlock
- added U_FG: BQ27Z561YPHR, gunnchos_structural:Block_SMD_10x10, symbol FuncBlock
- added U_HID: STM32F103C8T6, gunnchos_structural:Block_SMD_10x10, symbol FuncBlock
- added U_PD: TPS65987DDHRSHR, gunnchos_structural:Block_SMD_10x10, symbol FuncBlock
- added U_SE: SE050C1HQ1, gunnchos_structural:Block_SMD_10x10, symbol FuncBlock
- added U_WIFI: AP6275P, gunnchos_structural:Block_SMD_10x10, symbol FuncBlock
- added U_WWAN: RM520N-GL, gunnchos_structural:Block_SMD_10x10, symbol FuncBlock
Connections:
- new net CC1: SW_ABXY.2
- new net CC2: JS1.2
- new net GND: JSOM1.2
- new net HDMI0_TX: J_DISP.2
- new net I2C0_HID: U_SE.2
- new net I2S0: J_USD.2
- new net LCD_BL_PWM: U_WWAN.2
- new net LCD_RESET_L: U_HID.2
- new net MIPI_DPHY_TX: U_WIFI.2
- new net PCIE20_WWAN: J_AUDIO.2
- new net SDMMC: U_FG.2
- new net UART2_DBG: J_USBC.2
- new net USB20_HOST0_DM: U_PD.2
- new net USB30_SS: U_CHG.2
- new net VBAT: BT1.2
- new net VBUS_PD: J_DBG.2
- new net VCC_SYSIN: USOM1.2
- no-connect marks 0 -> 19
Other:
- company: gunnchOS3k / HARDWARE DESIGN RELEASE -> gunnchOS3k / CONTINUATION VII
- title: Handheld Hybrid SoM Carrier -> Handheld Hybrid SoM Carrier — Cont VII PUBLIC_PINOUT
