File: device_designs/handheld_hybrid/kicad/handheld_hybrid.kicad_sch (KiCad schematic)
At the start: 11 parts

Commit message: feat(family): exact MPNs and hardware design release candidates
Freeze orderable ADLINK COM-HPC-mMTL-155H-32G and Radxa NX5 RM121-D8E32,
verify RM520N-GL Sub-6 with no NTN claim, and deepen five-product EDA/CAD/mfg
packages as honest CANDIDATE releases under PHYSICAL_EXECUTION_FREEZE.

Co-authored-by: Cursor <cursoragent@cursor.com>
Parts:
- USOM1: value RK3588S-SoM-16GB -> RM121-D8E32
Other:
- company: gunnchOS3k / HARDWARE FAMILY DEPTH -> gunnchOS3k / HARDWARE DESIGN RELEASE
Changed lines of the file:
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@@
-(kicad_sch (version 20230121) (generator "family_depth_digital")
+(kicad_sch (version 20230121) (generator "hardware_design_release")
   (paper "A3")
   (title_block
@@
     (date "2026-08-08")
     (rev "0.2.0-dev")
-    (company "gunnchOS3k / HARDWARE FAMILY DEPTH")
+    (company "gunnchOS3k / HARDWARE DESIGN RELEASE")
     (comment 1 "RK3588S SoM + sustained game carrier")
     (comment 2 "ADR-FP-002 / ADR-HW-001")
@@
     (in_bom yes) (on_board yes) (dnp no)
     (property "Reference" "USOM1" (at 40 33 0) (effects (font (size 1.27 1.27))))
-    (property "Value" "RK3588S-SoM-16GB" (at 40 47 0) (effects (font (size 1.27 1.27))))
+    (property "Value" "RM121-D8E32" (at 40 47 0) (effects (font (size 1.27 1.27))))
     (property "Footprint" "" (at 40 40 0) (effects (font (size 1.27 1.27)) hide))
     (property "Datasheet" "" (at 40 40 0) (effects (font (size 1.27 1.27)) hide))

Commit message: feat(eda): Cont VI KiCad 10.0.5 CLI validation + PCB load fixes
Install path resolved; run ERC/DRC/Gerber/drill/PnP/STEP for all five boards.
Fix KiCad 10 PCB load blockers (unknown setup key on Student/DS-XL; odd
5-layer copper on Dock → 4-layer). Record RING_KICAD_CLI_VALIDATION_PASS
and honest per-board violation counts; NDA release posture unchanged.

Co-authored-by: Cursor <cursoragent@cursor.com>
Parts:
- added JS1, JS2: RKJXV122400D, symbol Device:R
- added JSOM1: SODIMM-260, SODIMM-260, symbol Device:R
- added J_AUDIO: I2S_HP_codec, symbol Device:R
- added J_DBG: UART2_3pin, symbol Device:R
- added J_USD: microSD_socket, symbol Device:R
- added SW_ABXY: tactile_ABXY_LR_DPAD, symbol Device:R
- BT1, U_SE: Evidence (none) -> PUBLIC_PINOUT
- J_DISP: value 7in_1080p_120Hz -> 7in_1080p_120Hz_IPS; Evidence (none) -> PUBLIC_PINOUT
- J_USBC: value USB_C_DP_Alt -> USB_C_receptacle; footprint (none) -> USB4085; Evidence (none) -> PUBLIC_PINOUT
- USOM1: footprint (none) -> SODIMM-260; Evidence (none) -> PUBLIC_PINOUT
- U_CHG: value BQ25895_or_BQ25792 -> BQ25895RTWR; Evidence (none) -> PUBLIC_PINOUT
- U_FG: value BQ27Z273 -> BQ27Z561YPHR; Evidence (none) -> PUBLIC_PINOUT
- U_HID: footprint (none) -> LQFP-48; Evidence (none) -> PUBLIC_PINOUT
- U_PD: value TPS65987_or_IP2726 -> TPS65987DDHRSHR; Evidence (none) -> PUBLIC_PINOUT
- U_WIFI: value AP6275P_or_AIC8800D -> AP6275P; Evidence (none) -> PUBLIC_PINOUT
- U_WWAN: footprint (none) -> M.2-B; Evidence (none) -> PUBLIC_PINOUT
Other:
- company: gunnchOS3k / HARDWARE DESIGN RELEASE -> gunnchOS3k / CONTINUATION VI
- title: Handheld Hybrid SoM Carrier -> Handheld Hybrid SoM Carrier — PUBLIC_PINOUT

Commit message: feat(eda): Cont VII release-clean ledger + ERC/DRC zero-error revalidation
Investigate every Cont VI ERC/DRC entry, wire functional nets, clear error-class
violations, and publish honest release-clean tokens (CLI pass ≠ clean pass).

Co-authored-by: Cursor <cursoragent@cursor.com>
Parts:
- removed BT1: 6000mAh_pack, symbol Device:R
- removed JS1, JS2: RKJXV122400D, symbol Device:R
- removed JSOM1: SODIMM-260, SODIMM-260, symbol Device:R
- removed J_AUDIO: I2S_HP_codec, symbol Device:R
- removed J_DBG: UART2_3pin, symbol Device:R
- removed J_DISP: 7in_1080p_120Hz_IPS, symbol Device:R
- removed J_USBC: USB_C_receptacle, USB4085, symbol Device:R
- removed J_USD: microSD_socket, symbol Device:R
- removed SW_ABXY: tactile_ABXY_LR_DPAD, symbol Device:R
- removed USOM1: RM121-D8E32, SODIMM-260, symbol Device:R
- removed U_CHG: BQ25895RTWR, symbol Device:R
- removed U_FG: BQ27Z561YPHR, symbol Device:R
- removed U_HID: STM32F103C8T6, LQFP-48, symbol Device:R
- removed U_PD: TPS65987DDHRSHR, symbol Device:R
- removed U_SE: SE050C1HQ1, symbol Device:R
- removed U_WIFI: AP6275P, symbol Device:R
- removed U_WWAN: RM520N-GL, M.2-B, symbol Device:R
- added BT1: 6000mAh_pack, gunnchos_structural:Block_SMD_10x10, symbol FuncBlock
- added JS1, JS2: RKJXV122400D, gunnchos_structural:Block_SMD_10x10, symbol FuncBlock
- added JSOM1: SODIMM-260, gunnchos_structural:Block_SMD_10x10, symbol FuncBlock
- added J_AUDIO: I2S_HP_codec, gunnchos_structural:Block_SMD_10x10, symbol FuncBlock
- added J_DBG: UART2_3pin, gunnchos_structural:Block_SMD_10x10, symbol FuncBlock
- added J_DISP: 7in_1080p_120Hz_IPS, gunnchos_structural:Block_SMD_10x10, symbol FuncBlock
- added J_USBC: USB_C_receptacle, gunnchos_structural:Block_SMD_10x10, symbol FuncBlock
- added J_USD: microSD_socket, gunnchos_structural:Block_SMD_10x10, symbol FuncBlock
- added SW_ABXY: tactile_ABXY_LR_DPAD, gunnchos_structural:Block_SMD_10x10, symbol FuncBlock
- added USOM1: RM121-D8E32, gunnchos_structural:Block_SMD_10x10, symbol FuncBlock
- added U_CHG: BQ25895RTWR, gunnchos_structural:Block_SMD_10x10, symbol FuncBlock
- added U_FG: BQ27Z561YPHR, gunnchos_structural:Block_SMD_10x10, symbol FuncBlock
- added U_HID: STM32F103C8T6, gunnchos_structural:Block_SMD_10x10, symbol FuncBlock
- added U_PD: TPS65987DDHRSHR, gunnchos_structural:Block_SMD_10x10, symbol FuncBlock
- added U_SE: SE050C1HQ1, gunnchos_structural:Block_SMD_10x10, symbol FuncBlock
- added U_WIFI: AP6275P, gunnchos_structural:Block_SMD_10x10, symbol FuncBlock
- added U_WWAN: RM520N-GL, gunnchos_structural:Block_SMD_10x10, symbol FuncBlock
Connections:
- net CC1: now also SW_ABXY.2
- net CC2: now also JS1.2
- net GND: now also JSOM1.2
- net HDMI0_TX: now also J_DISP.2
- net I2C0_HID: now also U_SE.2
- net I2S0: now also J_USD.2
- net LCD_BL_PWM: now also U_WWAN.2
- net LCD_RESET_L: now also U_HID.2
- net MIPI_DPHY_TX: now also U_WIFI.2
- net PCIE20_WWAN: now also J_AUDIO.2
- net SDMMC: now also U_FG.2
- net UART2_DBG: now also J_USBC.2
- net USB20_HOST0_DM: now also U_PD.2
- net USB30_SS: now also U_CHG.2
- net VBAT: now also BT1.2
- net VBUS_PD: now also J_DBG.2
- net VCC_SYSIN: now also USOM1.2
- no-connect marks 0 -> 19
Other:
- company: gunnchOS3k / CONTINUATION VI -> gunnchOS3k / CONTINUATION VII
- title: Handheld Hybrid SoM Carrier — PUBLIC_PINOUT -> Handheld Hybrid SoM Carrier — Cont VII PUBLIC_PINOUT

Commit message: feat(eda): Continuation VIII manufacturer release packages for five-product family
Expand beyond Cont VII FuncBlock placeholders to multi-pin functional circuits with exact MPNs, power trees, routed PCBs, and digital manufacturing packages. Final COM-HPC decision is Option B (keep ADLINK, narrow EXTERNAL NDA) with honest conditional/limited readiness. ERC/DRC errors are zero on all five boards under KiCad 10.0.5; PHYSICAL_EXECUTION_FREEZE remains active.

Co-authored-by: Cursor <cursoragent@cursor.com>
Parts:
- removed BT1: 6000mAh_pack, gunnchos_structural:Block_SMD_10x10, symbol FuncBlock
- removed JS1, JS2: RKJXV122400D, gunnchos_structural:Block_SMD_10x10, symbol FuncBlock
- removed JSOM1: SODIMM-260, gunnchos_structural:Block_SMD_10x10, symbol FuncBlock
- removed J_AUDIO: I2S_HP_codec, gunnchos_structural:Block_SMD_10x10, symbol FuncBlock
- removed J_DBG: UART2_3pin, gunnchos_structural:Block_SMD_10x10, symbol FuncBlock
- removed J_DISP: 7in_1080p_120Hz_IPS, gunnchos_structural:Block_SMD_10x10, symbol FuncBlock
- removed J_USBC: USB_C_receptacle, gunnchos_structural:Block_SMD_10x10, symbol FuncBlock
- removed J_USD: microSD_socket, gunnchos_structural:Block_SMD_10x10, symbol FuncBlock
- removed SW_ABXY: tactile_ABXY_LR_DPAD, gunnchos_structural:Block_SMD_10x10, symbol FuncBlock
- removed USOM1: RM121-D8E32, gunnchos_structural:Block_SMD_10x10, symbol FuncBlock
- removed U_CHG: BQ25895RTWR, gunnchos_structural:Block_SMD_10x10, symbol FuncBlock
- removed U_FG: BQ27Z561YPHR, gunnchos_structural:Block_SMD_10x10, symbol FuncBlock
- removed U_HID: STM32F103C8T6, gunnchos_structural:Block_SMD_10x10, symbol FuncBlock
- removed U_PD: TPS65987DDHRSHR, gunnchos_structural:Block_SMD_10x10, symbol FuncBlock
- removed U_SE: SE050C1HQ1, gunnchos_structural:Block_SMD_10x10, symbol FuncBlock
- removed U_WIFI: AP6275P, gunnchos_structural:Block_SMD_10x10, symbol FuncBlock
- removed U_WWAN: RM520N-GL, gunnchos_structural:Block_SMD_10x10, symbol FuncBlock
- added C1: CL05A104KA5NNNC, gunnchos_functional:C_0402, symbol C
- added C2: GRM188R60J106ME47D, gunnchos_functional:C_0402, symbol C
- added D1: APTD1608LCGCK, gunnchos_functional:LED_0603, symbol LED
- added DESD1: PESD5V0S1UL, gunnchos_functional:R_0402, symbol C
- added JSOM1: SODIMM-260, gunnchos_functional:Block_SMD_safe, symbol SODIMM260
- added JUSB1: TYPE-C-31-M-12, gunnchos_functional:Block_SMD_safe, symbol USB_C
- added R1: RC0402FR-0710KL, gunnchos_functional:R_0402, symbol R
- added R2: RC0402FR-071K0L, gunnchos_functional:R_0402, symbol R
- added U3V3: TPS62864, gunnchos_functional:Block_SMD_safe, symbol BUCK
- added UCHG1: BQ25895RTWR, gunnchos_functional:Block_SMD_safe, symbol CHARGER
- added UHID1: STM32F103C8T6, gunnchos_functional:Block_SMD_safe, symbol HID_MCU
- added UPD1: TPS65987DDHRSHR, gunnchos_functional:Block_SMD_safe, symbol PD_CTRL
Connections:
- net CC1: now also DESD1.1, JUSB1.A5 (CC1), UPD1.8 (3V3)
- net GND: now also C1.2, C2.2, D1.1 (K), DESD1.2, JSOM1.65 (HDMI0_TX2P), JUSB1.A7 (DM), U3V3.1 (VIN), UCHG1.4 (GND), UHID1.6 (SDA), UPD1.6 (SDA)
- net LCD_BL_PWM: now also JSOM1.185 (I2C0_SCL)
- net VBAT: now also UCHG1.3 (BAT)
- new net I2C_SCL: JSOM1.220 (LCD_BL_PWM), R1.2, UCHG1.1 (VBUS), UHID1.1 (VDD), UPD1.3 (CC2)
- new net I2C_SDA: JSOM1.238 (UART2_RX), UCHG1.2 (SYS), UHID1.2 (GND), UPD1.4 (GND)
- new net LED_A: D1.2 (A), R2.2
- new net SOM_VIN: JSOM1.227 (SDMMC_CMD)
- new net UART_RX: JSOM1.187 (I2C0_SDA)
- new net UART_TX: JSOM1.63 (HDMI0_TX2N)
- new net USB_DM: JSOM1.219 (SDMMC_D0), UHID1.4 (USB_DM)
- new net USB_DP: JSOM1.126 (LCD_RESET_L), UHID1.3 (USB_DP)
- new net VBUS: JUSB1.B5 (CC2), UCHG1.5 (SCL), UPD1.7 (VSYS)
- new net VDD_3V3: C1.1, R1.1, R2.1, U3V3.2 (EN), U3V3.4 (VOUT), UHID1.5 (SCL), UPD1.2 (CC1)
- new net VSYS: C2.1, U3V3.3 (GND), UCHG1.6 (SDA), UPD1.1 (VBUS)
- no-connect marks 19 -> 11
Other:
- note added: "Cont VIII functional schematic — multi-pin symbols + exact MPNs (not FuncBlock placeholders)."
- note added: "Revision 0.5.0-cont-viii."
- note added: "SI notes encoded on PCB stackup/Dwgs — no SI simulation claimed."
- company: gunnchOS3k / CONTINUATION VII -> gunnchOS3k / CONTINUATION VIII
- title: Handheld Hybrid SoM Carrier — Cont VII PUBLIC_PINOUT -> Handheld Hybrid SoM Carrier — Cont VIII PUBLIC_PINOUT
