File: device_designs/handheld_hybrid/kicad/sheets/sodimm_other.kicad_sch (KiCad schematic)
At the start: 1 part

Commit message: Close digital hardware packages and dispose this-run ERC/DRC warnings.
Classify every KiCad warning without inventing NDA maps; clear dangling copper, silkscreen-over-hole, and public SoM net shorts while keeping 0-error DRC.

Co-authored-by: Cursor <cursoragent@cursor.com>
Connections:
- net SOM_4A1: no longer JS_OTHER.24 (MIPI_DPHY0_RX_D0P)
- net SOM_MIPI_DPHY0_RX_D0N: no longer JS_OTHER.230 (HP_DET_L), JS_OTHER.237 (POWER-EN)
- net SOM_MIPI_DPHY0_RX_D0P: no longer JS_OTHER.226 (4A1), JS_OTHER.235 (BBAT), JS_OTHER.240 (SLEEP-WAKE)
- new net SOM_BBAT: JS_OTHER.24 (MIPI_DPHY0_RX_D0P)
- new net SOM_MIPI_DPHY0_RX_D1N: JS_OTHER.230 (HP_DET_L), JS_OTHER.237 (POWER-EN)
- new net SOM_MIPI_DPHY0_RX_D1P: JS_OTHER.240 (SLEEP-WAKE)
- new net SOM_MIPI_DPHY1_RX_D2P: JS_OTHER.226 (4A1), JS_OTHER.235 (BBAT)
Changed lines of the file:
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@@
       (effects (font (size 1.27 1.27)) hide))
   )
-  (wire (pts (xy 59.68 127.94000000000001) (xy 59.68 125.4))
-    (stroke (width 0) (type default)))
   (global_label "SOM_MIPI_DPHY0_RX_D0P" (shape input) (at 100.32 127.94000000000001 90) (fields_autoplaced)
     (effects (font (size 1.27 1.27)) (justify left))
@@
       (effects (font (size 1.27 1.27)) hide))
   )
-  (wire (pts (xy 100.32 127.94000000000001) (xy 100.32 125.4))
-    (stroke (width 0) (type default)))
   (global_label "SOM_MIPI_DPHY0_RX_D1N" (shape input) (at 59.68 125.4 90) (fields_autoplaced)
     (effects (font (size 1.27 1.27)) (justify left))
@@
       (effects (font (size 1.27 1.27)) hide))
   )
-  (wire (pts (xy 100.32 125.4) (xy 100.32 122.86))
-    (stroke (width 0) (type default)))
   (global_label "SOM_MIPI_DPHY1_RX_D2N" (shape input) (at 57.14 120.32 180) (fields_autoplaced)
     (effects (font (size 1.27 1.27)) (justify left))
@@
       (effects (font (size 1.27 1.27)) hide))
   )
-  (wire (pts (xy 100.32 74.6) (xy 100.32 77.14))
-    (stroke (width 0) (type default)))
   (global_label "SOM_POWER-EN" (shape input) (at 59.68 72.05999999999999 270) (fields_autoplaced)
     (effects (font (size 1.27 1.27)) (justify left))
@@
       (effects (font (size 1.27 1.27)) hide))
   )
-  (wire (pts (xy 59.68 72.05999999999999) (xy 59.68 74.6))
-    (stroke (width 0) (type default)))
   (global_label "SOM_SLEEP-WAKE" (shape input) (at 100.32 72.05999999999999 270) (fields_autoplaced)
     (effects (font (size 1.27 1.27)) (justify left))
@@
       (effects (font (size 1.27 1.27)) hide))
   )
-  (wire (pts (xy 100.32 72.05999999999999) (xy 100.32 74.6))
-    (stroke (width 0) (type default)))
   (sheet_instances
     (path "/" (page "1"))
