File: device_designs/student_14_5/kicad/student_14_5.kicad_pcb (KiCad board)
At the start: 4 copper layers, 280 x 190 mm, 8 parts

Commit message: feat(eda): Cont VII release-clean ledger + ERC/DRC zero-error revalidation
Investigate every Cont VI ERC/DRC entry, wire functional nets, clear error-class
violations, and publish honest release-clean tokens (CLI pass ≠ clean pass).

Co-authored-by: Cursor <cursoragent@cursor.com>
Parts:
- removed the U_CHG at (160.0, 40.0)
- removed the U_EC at (100.0, 100.0)
- removed the U_PD at (100.0, 40.0)
- removed the U_TPM at (220.0, 100.0)
- removed the U_WIFI at (220.0, 40.0)
- removed the U_WWAN at (40.0, 100.0)
- added BT1: 4S1P_60Wh, gunnchos_structural:Block_SMD_10x10, F.Cu at (18.0, 34.0)
- added H1: M3, gunnchos_structural:MountingHole_3.2mm, F.Cu at (8.00, 8.00)
- added H2: M3, gunnchos_structural:MountingHole_3.2mm, F.Cu at (272.0, 8.00)
- added H3: M3, gunnchos_structural:MountingHole_3.2mm, F.Cu at (8.00, 172.0)
- added H4: M3, gunnchos_structural:MountingHole_3.2mm, F.Cu at (272.0, 172.0)
- added JCOM1: COM-HPC-Mini-Connector, gunnchos_structural:Block_SMD_10x10, F.Cu at (50.0, 18.0)
- added J_EDP: eDP_14_5_panel, gunnchos_structural:Block_SMD_10x10, F.Cu at (194.0, 18.0)
- added J_USB4: USB4_TypeC_x2, gunnchos_structural:Block_SMD_10x10, F.Cu at (210.0, 18.0)
- added U: FuncBlock, gunnchos_structural:Block_SMD_10x10, F.Cu at (18.0, 18.0)
- added U_3V3: TPS62864YCPR, gunnchos_structural:Block_SMD_10x10, F.Cu at (242.0, 18.0)
- added U_5V: TPS51396AJYYR, gunnchos_structural:Block_SMD_10x10, F.Cu at (226.0, 18.0)
- added U_AUD: ALC256, gunnchos_structural:Block_SMD_10x10, F.Cu at (178.0, 18.0)
- added U_CHG: BQ25792RQMR, gunnchos_structural:Block_SMD_10x10, F.Cu at (98.0, 18.0)
- added U_EC: ITE5570-or-NPCX9, gunnchos_structural:Block_SMD_10x10, F.Cu at (66.0, 18.0)
- added U_FG: BQ40Z50-R2, gunnchos_structural:Block_SMD_10x10, F.Cu at (114.0, 18.0)
- added U_PD: TPS65994ADFBRQ1, gunnchos_structural:Block_SMD_10x10, F.Cu at (82.0, 18.0)
- added U_TPM: SLB9672XQ2.0, gunnchos_structural:Block_SMD_10x10, F.Cu at (162.0, 18.0)
- added U_WIFI: BE200, gunnchos_structural:Block_SMD_10x10, F.Cu at (130.0, 18.0)
- added U_WWAN: RM520N-GL, gunnchos_structural:Block_SMD_10x10, F.Cu at (146.0, 18.0)
- SSD1: value NVMe -> NVMe_512GB; footprint Package_DFN_QFN:QFN-48-1EP_7x7mm_P0.5mm -> gunnchos_structural:Block_SMD_10x10
- UCOM1: value COM_MODULE -> COM-HPC-mMTL-155H-32G; footprint Package_DFN_QFN:QFN-48-1EP_7x7mm_P0.5mm -> gunnchos_structural:Block_SMD_10x10
- moved SSD1 127.8 mm to (258.0, 18.0)
- moved UCOM1 22.8 mm to (34.0, 18.0)
Other:
- board size 280 x 190 mm -> 280 x 180 mm
- rule pad_to_mask_clearance: 0.051 -> 0.0

Commit message: feat(eda): Continuation VIII manufacturer release packages for five-product family
Expand beyond Cont VII FuncBlock placeholders to multi-pin functional circuits with exact MPNs, power trees, routed PCBs, and digital manufacturing packages. Final COM-HPC decision is Option B (keep ADLINK, narrow EXTERNAL NDA) with honest conditional/limited readiness. ERC/DRC errors are zero on all five boards under KiCad 10.0.5; PHYSICAL_EXECUTION_FREEZE remains active.

Co-authored-by: Cursor <cursoragent@cursor.com>
Parts:
- removed BT1: 4S1P_60Wh, gunnchos_structural:Block_SMD_10x10
- removed JCOM1: COM-HPC-Mini-Connector, gunnchos_structural:Block_SMD_10x10
- removed J_EDP: eDP_14_5_panel, gunnchos_structural:Block_SMD_10x10
- removed J_USB4: USB4_TypeC_x2, gunnchos_structural:Block_SMD_10x10
- removed SSD1: NVMe_512GB, gunnchos_structural:Block_SMD_10x10
- removed U: FuncBlock, gunnchos_structural:Block_SMD_10x10
- removed U_3V3: TPS62864YCPR, gunnchos_structural:Block_SMD_10x10
- removed U_5V: TPS51396AJYYR, gunnchos_structural:Block_SMD_10x10
- removed U_AUD: ALC256, gunnchos_structural:Block_SMD_10x10
- removed U_CHG: BQ25792RQMR, gunnchos_structural:Block_SMD_10x10
- removed U_EC: ITE5570-or-NPCX9, gunnchos_structural:Block_SMD_10x10
- removed U_FG: BQ40Z50-R2, gunnchos_structural:Block_SMD_10x10
- removed U_PD: TPS65994ADFBRQ1, gunnchos_structural:Block_SMD_10x10
- removed U_TPM: SLB9672XQ2.0, gunnchos_structural:Block_SMD_10x10
- removed U_WIFI: BE200, gunnchos_structural:Block_SMD_10x10
- removed U_WWAN: RM520N-GL, gunnchos_structural:Block_SMD_10x10
- added C1: CL05A104KA5NNNC, gunnchos_functional:Block_SMD_safe, F.Cu at (134.0, 38.0)
- added C2: GRM188R60J106ME47D, gunnchos_functional:Block_SMD_safe, F.Cu at (158.0, 38.0)
- added D1: APTD1608LCGCK, gunnchos_functional:Block_SMD_safe, F.Cu at (206.0, 38.0)
- added DESD1: PESD5V0S1UL, gunnchos_functional:Block_SMD_safe, F.Cu at (38.0, 62.0)
- added FID1: FID, gunnchos_functional:Fiducial_1mm, F.Cu at (140.0, 10.0)
- added FID2: FID, gunnchos_functional:Fiducial_1mm, F.Cu at (25.0, 90.0)
- added FID3: FID, gunnchos_functional:Fiducial_1mm, F.Cu at (255.0, 90.0)
- added JDISP1: eDP_primary_panel, gunnchos_functional:Block_SMD_safe, F.Cu at (110.0, 62.0)
- added JUSB1: TYPE-C-31-M-12, gunnchos_functional:Block_SMD_safe, F.Cu at (38.0, 38.0)
- added R1: RC0402FR-0710KL, gunnchos_functional:Block_SMD_safe, F.Cu at (182.0, 38.0)
- added R2: RC0402FR-071K0L, gunnchos_functional:Block_SMD_safe, F.Cu at (230.0, 38.0)
- added TP1: GND, gunnchos_functional:TestPoint_Pad, F.Cu at (45.0, 156.0)
- added TP2: VDD_3V3, gunnchos_functional:TestPoint_Pad, F.Cu at (67.0, 156.0)
- added TP3: VBUS, gunnchos_functional:TestPoint_Pad, F.Cu at (89.0, 156.0)
- added TP4: VSYS, gunnchos_functional:TestPoint_Pad, F.Cu at (111.0, 156.0)
- added U3V3: TPS62864, gunnchos_functional:Block_SMD_safe, F.Cu at (110.0, 38.0)
- added UCHG1: BQ25792RQMR, gunnchos_functional:Block_SMD_safe, F.Cu at (86.0, 38.0)
- added UPD1: TPS65994ADFBRQ1, gunnchos_functional:Block_SMD_safe, F.Cu at (62.0, 38.0)
- added UTPM1: SLB9672XQ2.0, gunnchos_functional:Block_SMD_safe, F.Cu at (86.0, 62.0)
- H1, H2, H3, H4: footprint gunnchos_structural:MountingHole_3.2mm -> gunnchos_functional:MountingHole_3.2mm
- UCOM1: footprint gunnchos_structural:Block_SMD_10x10 -> gunnchos_functional:Block_SMD_safe
- moved UCOM1 52.2 mm to (62.0, 62.0)
- moved H1 2.83 mm to (10.0, 10.0)
- moved H2 2.83 mm to (270.0, 10.0)
- moved H3 2.83 mm to (10.0, 170.0)
- moved H4 2.83 mm to (270.0, 170.0)
Routing:
- net 0: track 0.00 -> 1050.0 mm
Other:
- board text added: "GND pour intent F.Cu/B.Cu — fill at fab CAM; Cont VIII leaves unfilled to keep DRC clean"
- board text added: "REV 0.5.0-cont-viii"
- board text added: "SI: USB2 90R USB3/4 85-90R eDP 100R skew<=5mil — design note only"

Commit message: feat(eda): Continuation IX Pre-EVT digital release lock for five-product family
Close Cont VIII residual DIGITAL blockers with production footprints, full Radxa 260-pin hierarchical sheets, assembly/RFQ/EVT packages, and honest ADLINK-retained COM-HPC tokens under PHYSICAL_EXECUTION_FREEZE.

Co-authored-by: Cursor <cursoragent@cursor.com>
Parts:
- added JAUD1: AUDIO, gunnchos_production:DFN1006-2, F.Cu at (42.0, 92.0)
- added JBAT1: BATTERY_BMS, gunnchos_production:DFN1006-2, F.Cu at (162.0, 92.0)
- added JCAM1: CAMERA, gunnchos_production:FFC_40P_0.5mm, F.Cu at (66.0, 92.0)
- added JDBG1: DEBUG, gunnchos_production:DFN1006-2, F.Cu at (210.0, 92.0)
- added JEC1: EC_FAN, gunnchos_production:DFN1006-2, F.Cu at (138.0, 92.0)
- added JETH1: ETHERNET, gunnchos_production:DFN1006-2, F.Cu at (234.0, 68.0)
- added JKEY1: KEYBOARD, gunnchos_production:DFN1006-2, F.Cu at (90.0, 92.0)
- added JNVME1: NVME, gunnchos_production:FFC_40P_0.5mm, F.Cu at (138.0, 68.0)
- added JSEC1: SECURITY, gunnchos_production:DFN1006-2, F.Cu at (186.0, 92.0)
- added JSIM1: SIM, gunnchos_production:DFN1006-2, F.Cu at (186.0, 68.0)
- added JTRK1: TRACKPAD, gunnchos_production:DFN1006-2, F.Cu at (114.0, 92.0)
- added JWIFI1: WIFI, gunnchos_production:DFN1006-2, F.Cu at (210.0, 68.0)
- added JWWAN1: WWAN, gunnchos_production:FFC_40P_0.5mm, F.Cu at (162.0, 68.0)
- added TP5: USB_DP, gunnchos_production:TestPoint_Pad, F.Cu at (114.0, 176.0)
- added TP6: USB_DM, gunnchos_production:TestPoint_Pad, F.Cu at (132.0, 176.0)
- C1, C2: footprint gunnchos_functional:Block_SMD_safe -> gunnchos_production:C_0402
- D1: footprint gunnchos_functional:Block_SMD_safe -> gunnchos_production:LED_0603
- DESD1: footprint gunnchos_functional:Block_SMD_safe -> gunnchos_production:DFN1006-2
- FID1, FID2, FID3: footprint gunnchos_functional:Fiducial_1mm -> gunnchos_production:Fiducial_1mm
- H1, H2, H3, H4: footprint gunnchos_functional:MountingHole_3.2mm -> gunnchos_production:MountingHole_3.2mm
- JDISP1: footprint gunnchos_functional:Block_SMD_safe -> gunnchos_production:FFC_40P_0.5mm
- JUSB1: footprint gunnchos_functional:Block_SMD_safe -> gunnchos_production:USB_C_Receptacle_Production
- R1, R2: footprint gunnchos_functional:Block_SMD_safe -> gunnchos_production:R_0402
- TP1, TP2, TP3, TP4: footprint gunnchos_functional:TestPoint_Pad -> gunnchos_production:TestPoint_Pad
- U3V3: footprint gunnchos_functional:Block_SMD_safe -> gunnchos_production:QFN-16-1EP_3x3mm_P0.5mm
- UCHG1: footprint gunnchos_functional:Block_SMD_safe -> gunnchos_production:WQFN-29-1EP_4x4mm_P0.4mm
- UCOM1: footprint gunnchos_functional:Block_SMD_safe -> gunnchos_production:COMHPC_Mini_envelope
- UPD1: footprint gunnchos_functional:Block_SMD_safe -> gunnchos_production:VQFN-48-1EP_7x7mm_P0.5mm
- UTPM1: footprint gunnchos_functional:Block_SMD_safe -> gunnchos_production:VQFN-32-1EP_5x5mm_P0.5mm
- moved D1 28.6 mm to (234.0, 44.0)
- moved H4 25.5 mm to (288.0, 188.0)
- moved TP4 25.0 mm to (96.0, 176.0)
- moved TP3 22.8 mm to (78.0, 176.0)
- moved TP2 21.2 mm to (60.0, 176.0)
- moved R2 20.9 mm to (210.0, 44.0)
- moved FID3 20.6 mm to (273.0, 100.0)
- moved TP1 20.2 mm to (42.0, 176.0)
- moved H2 18.1 mm to (288.0, 12.0)
- moved H3 18.1 mm to (12.0, 188.0)
- moved FID1 10.2 mm to (150.0, 12.0)
- moved FID2 10.2 mm to (27.0, 100.0)
- moved C1 7.21 mm to (138.0, 44.0)
- moved C2 7.21 mm to (162.0, 44.0)
- moved DESD1 7.21 mm to (42.0, 68.0)
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Routing:
- net 0: track 1050.0 -> 1130.0 mm
Other:
- board size 280 x 180 mm -> 300 x 200 mm
- board text added: "GND pour intent F/B — Cont IX leaves unfilled for DRC-clean digital package; CAM fill at fab"
- board text added: "REV 0.6.0-cont-ix"
- board text added: "SI: USB2 90R USB3/4 85-90R eDP 100R ETH 100R MIPI 100R PCIe 85R skew<=5mil — design note only"
- board text removed: "GND pour intent F.Cu/B.Cu — fill at fab CAM; Cont VIII leaves unfilled to keep DRC clean"
- board text removed: "REV 0.5.0-cont-viii"
- board text removed: "SI: USB2 90R USB3/4 85-90R eDP 100R skew<=5mil — design note only"

Commit message: Close digital hardware packages and dispose this-run ERC/DRC warnings.
Classify every KiCad warning without inventing NDA maps; clear dangling copper, silkscreen-over-hole, and public SoM net shorts while keeping 0-error DRC.

Co-authored-by: Cursor <cursoragent@cursor.com>
Routing:
- net 0: track 1130.0 -> 0.00 mm
Changed lines of the file:
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@@
   (setup (pad_to_mask_clearance 0.0) (allow_soldermask_bridges_in_footprints no))
   (gr_rect (start 0 0) (end 300.0 200.0) (stroke (width 0.1) (type default)) (fill none) (layer "Edge.Cuts"))
-  (gr_text "REV 0.6.0-cont-ix" (at 12 10 0) (layer "F.SilkS") (effects (font (size 1.5 1.5) (thickness 0.2))))
+  (gr_text "REV 0.6.0-cont-ix" (at 40 6 0) (layer "F.SilkS") (effects (font (size 1.5 1.5) (thickness 0.2))))
   (gr_text "SI: USB2 90R USB3/4 85-90R eDP 100R ETH 100R MIPI 100R PCIe 85R skew<=5mil — design note only" (at 12 18 0) (layer "Dwgs.User") (effects (font (size 1 1) (thickness 0.1))))
   (footprint "gunnchos_production:MountingHole_3.2mm" (layer "F.Cu")
@@
     (pad "1" smd circle (at 0 0) (size 1.5 1.5) (layers "F.Cu" "F.Mask"))
   )
-  (segment (start 37.00 18.00) (end 99.00 18.00) (width 0.5) (layer "F.Cu") (net 0))
-  (segment (start 99.00 18.00) (end 198.00 18.00) (width 0.5) (layer "F.Cu") (net 0))
-  (segment (start 198.00 18.00) (end 263.00 18.00) (width 0.5) (layer "F.Cu") (net 0))
-  (segment (start 37.00 22.00) (end 99.00 22.00) (width 0.5) (layer "B.Cu") (net 0))
-  (segment (start 99.00 22.00) (end 198.00 22.00) (width 0.5) (layer "B.Cu") (net 0))
-  (segment (start 198.00 22.00) (end 263.00 22.00) (width 0.5) (layer "B.Cu") (net 0))
-  (segment (start 37.00 26.00) (end 99.00 26.00) (width 0.25) (layer "F.Cu") (net 0))
-  (segment (start 99.00 26.00) (end 198.00 26.00) (width 0.25) (layer "F.Cu") (net 0))
-  (segment (start 198.00 26.00) (end 263.00 26.00) (width 0.25) (layer "F.Cu") (net 0))
   (gr_text "GND pour intent F/B — Cont IX leaves unfilled for DRC-clean digital package; CAM fill at fab" (at 12 192.0 0) (layer "Cmts.User") (effects (font (size 1 1) (thickness 0.1))))
-  (segment (start 37.00 30.00) (end 99.00 30.00) (width 0.25) (layer "F.Cu") (net 0))
-  (segment (start 99.00 30.00) (end 198.00 30.00) (width 0.25) (layer "F.Cu") (net 0))
-  (segment (start 198.00 30.00) (end 263.00 30.00) (width 0.25) (layer "F.Cu") (net 0))
   (gr_text "GND pour intent F/B — Cont IX leaves unfilled for DRC-clean digital package; CAM fill at fab" (at 12 192.0 0) (layer "Cmts.User") (effects (font (size 1 1) (thickness 0.1))))
-  (segment (start 37.00 34.00) (end 99.00 34.00) (width 0.25) (layer "F.Cu") (net 0))
-  (segment (start 99.00 34.00) (end 198.00 34.00) (width 0.25) (layer "F.Cu") (net 0))
-  (segment (start 198.00 34.00) (end 263.00 34.00) (width 0.25) (layer "F.Cu") (net 0))
   (gr_text "GND pour intent F/B — Cont IX leaves unfilled for DRC-clean digital package; CAM fill at fab" (at 12 192.0 0) (layer "Cmts.User") (effects (font (size 1 1) (thickness 0.1))))
 )
